File: MAX232.kicad_sch (KiCad schematic)
At the start: 6 parts, among them U1 MAX232

Commit message: Fabricated 10/10/23
Connections:
- net GND: now also C4.1; no longer C4.2
- net at U1.6 (VS-): now also C4.2; no longer C4.1
Other:
- moved on the sheet: C4
Changed lines of the file:
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@@
     )
   )
-  (symbol (lib_id "Device:C_Polarized") (at 173.99 100.33 0) (unit 1)
+  (symbol (lib_id "Device:C_Polarized") (at 173.99 100.33 180) (unit 1)
     (in_bom yes) (on_board yes) (dnp no)
-    (property "Reference" "C4" (at 174.625 97.79 0)
+    (property "Reference" "C4" (at 173.355 102.87 0)
       (effects (font (size 1.27 1.27)) (justify left))
     )
-    (property "Value" "1µF" (at 174.625 102.87 0)
+    (property "Value" "1µF" (at 173.355 97.79 0)
       (effects (font (size 1.27 1.27)) (justify left))
     )
-    (property "Footprint" "Capacitor_SMD:C_1206_3216Metric_Pad1.33x1.80mm_HandSolder" (at 174.9552 104.14 0)
+    (property "Footprint" "Capacitor_SMD:C_1206_3216Metric_Pad1.33x1.80mm_HandSolder" (at 173.0248 96.52 0)
       (effects (font (size 1.27 1.27)) hide)
     )

Commit message: Updated to kicad 9
Parts:
- renumbered C5 to C10, C2 to C11, C4 to C12, C3 to C13, C1 to C9
